File: F1C200S-HomeAssistant-Board/F1C200S-HomeAssistant-Board.kicad_pcb (KiCad board)
At the start: 2 copper layers, 85 x 56 mm, 93 parts, among them J1 Conn_01x02, J2 Conn_01x20, J3 CORE2_LCD_FPC_10P, J4 Conn_01x20, SW1 TS-1101-C-W, U1 F1C200S, U2 EA3036C, U3 XC6206P302MR, U4 GT-USB-7010ASV, U5 CH340C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

Commit message: docs: 更新制作文件
Parts:
- added REF**: OSHW-Symbol_6.7x6mm_SilkScreen, Symbol:OSHW-Symbol_6.7x6mm_SilkScreen, F.Cu at (61.9, 140.6)
